Commit message: fix: arm_driver dual gripper IDs and arm_joint3 axis/offset/limits
- arm_driver: gripper_id -> gripper_ids [27, 28] with directions [1.0, -1.0]
- arm_driver: gripper_offsets (per-servo), Current_Limit clamping on init
- arm_driver: detailed error messages per ID/register in init_motors
- arm_gripper_driver.yaml: gripper_ids/directions/offsets updated
- arm_gripper_driver.yaml: arm_offsets[2] = -2.4222 for joint3 zero-point
- sekirei.urdf: arm_joint3 axis 0 1 0 -> 0 -1 0, limits -3.14~3.14

Co-Authored-By: Claude Sonnet 4.6 <noreply@anthropic.com>

File: main_ws/src/bringup/urdf/sekirei.urdf (robot description, URDF)
Before this commit: robot sekirei, 13 links, 12 joints
Joints:
- joint arm_joint3: axis 0 1 0 -> 0 -1 0; limit lower=0 upper=3.14 effort=5 velocity=1.571 -> lower=-3.14 upper=3.14 effort=5 velocity=1.571

Commit message: fix: arm_joint3 direction inversion for worm gear (servo 23)
ウォームギアによりURDF関節方向とサーボ回転方向が逆のため、
グリッパーと同パターンの arm_directions パラメータを追加。
servo 23 (arm_joint3) に direction=-1.0 を設定。
sekirei.urdf の arm_joint3 axis を xacro と統一 (0 1 0)。
pre-commit の cargo-clippy をワークスペース未ビルド時スキップに変更。

Co-Authored-By: Claude Sonnet 4.6 <noreply@anthropic.com>

File: main_ws/src/bringup/urdf/sekirei.urdf (robot description, URDF)
Before this commit: robot sekirei, 13 links, 12 joints
Joints:
- joint arm_joint3: axis 0 -1 0 -> 0 1 0
