Commit message: flipper moved

File: main_ws/src/bringup/urdf/sekirei.urdf (robot description, URDF)
Before this commit: robot sekirei, 13 links, 12 joints
Joints:
- joint arm_joint3: limit lower=-3.14 upper=3.14 effort=5 velocity=1.571 -> lower=-0.72 upper=3.14 effort=5 velocity=1.571

Commit message: arm

File: main_ws/src/bringup/urdf/sekirei.urdf (robot description, URDF)
Before this commit: robot sekirei, 13 links, 12 joints
Joints:
- joint arm_joint3: axis 0 1 0 -> 0 -1 0
- joint arm_joint4: axis 0 1 0 -> 0 -1 0

File: main_ws/src/control/moveit/urdf/sekirei_moveit.xacro (robot description, xacro)
@@ -105,5 +105,5 @@
   <joint name="arm_joint3" type="revolute">
     <origin xyz="0.45 0.007 0.084" rpy="0 0 0"/>
-    <axis xyz="0 1 0"/>
+    <axis xyz="0 -1 0"/>
     <parent link="arm2_link"/>
     <child link="arm3_link"/>
@@ -130,5 +130,5 @@
   <joint name="arm_joint4" type="revolute">
     <origin xyz="-0.5 0.012 0" rpy="0 0 0"/>
-    <axis xyz="0 1 0"/>
+    <axis xyz="0 -1 0"/>
     <parent link="arm3_link"/>
     <child link="arm4_link"/>
