Commit message: feat: H264カメラ配信・シミュレーション修正・WebRTC削除・RoboCup認識実装
- camera: v4l2_camera + ffmpeg_image_transport (libx264) → foxglove_msgs/CompressedVideo
- simulation: URDF物理設定・Gazeboプラグイン・headlessモード・TimerAction遅延を修正
- webrtc: ros2_webrtc / gst_webrtc_operator / h264_republisher を削除
- audio: operator_ws に audio_bridge シンボリックリンク追加
- perception: robo_map_exporter (PLY/PNG/CSV), poi_writer 汎用化, qr_detector POI統合
- launch: use_lidar/use_camera/use_arm/use_flipper/use_imu フラグ追加
- ci: cachix continue-on-error 対応, pyproject.toml (ruff/black) 追加
- topology: system/network mermaid 図を現状に合わせ更新

Co-Authored-By: Claude Sonnet 4.6 <noreply@anthropic.com>

File: main_ws/src/bringup/urdf/robot.urdf.xacro (robot description, xacro)
@@ -12,6 +12,18 @@
   <material name="white"><color rgba="1 1 1 1"/></material>
   <!-- ======================== Base ======================== -->
+  <link name="base_footprint"/>
+  <joint name="base_footprint_joint" type="fixed">
+    <parent link="base_footprint"/>
+    <child link="base_link"/>
+    <origin xyz="0 0 ${wheel_radius}"/>
+  </joint>
   <link name="base_link">
     <visual><geometry><box size="${base_length} ${base_width} ${base_height}"/></geometry><material name="silver"/></visual>
+    <collision><geometry><box size="${base_length} ${base_width} ${base_height}"/></geometry></collision>
+    <inertial>
+      <mass value="15.0"/>
+      <origin xyz="0 0 0"/>
+      <inertia ixx="0.175" ixy="0" ixz="0" iyy="0.600" iyz="0" izz="0.725"/>
+    </inertial>
   </link>
   <!-- Flippers (RPY based on Mesh Z-axis as length) -->
@@ -60,3 +72,120 @@
   </link>
   <joint name="arm_joint6" type="revolute"><origin xyz="0.07425 0 -0.03"/><axis xyz="1 0 0"/><parent link="arm5_link"/><child link="arm6_link"/><limit effort="5" lower="-3.14" upper="3.14" velocity="1.571"/></joint>
+  <!-- ======================== Simulation: Drive Wheels ======================== -->
+  <!-- クローラを diff_drive で近似する仮想ホイール (シミュレーション専用) -->
+  <xacro:macro name="drive_wheel" params="name y_offset">
+    <link name="${name}">
+      <visual>
+        <origin rpy="${pi/2} 0 0"/>
+        <geometry><cylinder radius="${wheel_radius}" length="${wheel_width}"/></geometry>
+        <material name="silver"/>
+      </visual>
+      <collision>
+        <origin rpy="${pi/2} 0 0"/>
+        <geometry><cylinder radius="${wheel_radius}" length="${wheel_width}"/></geometry>
+      </collision>
+      <inertial>
+        <mass value="1.0"/>
+        <inertia ixx="0.001" ixy="0" ixz="0" iyy="0.002" iyz="0" izz="0.001"/>
+      </inertial>
+    </link>
+    <joint name="${name}_joint" type="continuous">
+      <parent link="base_link"/>
+      <child link="${name}"/>
+      <origin xyz="0 ${y_offset} ${-base_height/2}"/>
+      <axis xyz="0 1 0"/>
+    </joint>
+  </xacro:macro>
+  <xacro:drive_wheel name="left_wheel"  y_offset="${track_width/2}"/>
+  <xacro:drive_wheel name="right_wheel" y_offset="${-track_width/2}"/>
+  <!-- ======================== Simulation: Sensors ======================== -->
+  <link name="velodyne">
+    <visual>
+      <geometry><cylinder radius="0.05" length="0.07"/></geometry>
+      <material name="silver"/>
+    </visual>
+    <collision>
+      <geometry><cylinder radius="0.05" length="0.07"/></geometry>
+    </collision>
+    <inertial>
+      <mass value="0.8"/>
+      <inertia ixx="0.001" ixy="0" ixz="0" iyy="0.001" iyz="0" izz="0.001"/>
+    </inertial>
+  </link>
+  <joint name="velodyne_joint" type="fixed">
+    <parent link="base_link"/>
+    <child link="velodyne"/>
+    <origin xyz="0.15 0 ${base_height/2 + 0.05}"/>
+  </joint>
+  <link name="imu_link"/>
+  <joint name="imu_joint" type="fixed">
+    <parent link="base_link"/>
+    <child link="imu_link"/>
+    <origin xyz="0 0 0"/>
+  </joint>
+  <!-- ======================== Gazebo Plugins ======================== -->
+  <!-- DiffDrive: /cmd_vel → 走行、/odom → オドメトリ出力 -->
+  <gazebo>
+    <plugin filename="gz-sim-diff-drive-system"
+            name="gz::sim::systems::DiffDrive">
+      <left_joint>left_wheel_joint</left_joint>
+      <right_joint>right_wheel_joint</right_joint>
+      <wheel_separation>${track_width}</wheel_separation>
+      <wheel_radius>${wheel_radius}</wheel_radius>
+      <topic>cmd_vel</topic>
+      <odom_topic>odom</odom_topic>
+      <frame_id>odom</frame_id>
+      <child_frame_id>base_footprint</child_frame_id>
+      <odom_publish_frequency>50</odom_publish_frequency>
+      <!-- TFはodom_tf_bridge.pyが発行するためここでは無効 -->
+      <publish_odom_tf>false</publish_odom_tf>
+    </plugin>
+  </gazebo>
+  <!-- JointStatePublisher: アーム・フリッパの状態を/joint_statesへ -->
+  <gazebo>
+    <plugin filename="gz-sim-joint-state-publisher-system"
+            name="gz::sim::systems::JointStatePublisher">
+      <topic>joint_states</topic>
+      <update_rate>50</update_rate>
+    </plugin>
+  </gazebo>
+  <!-- LiDAR (GPU必須。nixGL環境またはGPU搭載マシンのみ有効) -->
+  <gazebo reference="velodyne">
+    <sensor name="vlp16" type="gpu_lidar">
+      <topic>velodyne_points</topic>
+      <update_rate>10</update_rate>
+      <gz_frame_id>velodyne</gz_frame_id>
+      <lidar>
+        <scan>
+          <horizontal>
+            <samples>1800</samples>
+            <resolution>1</resolution>
+            <min_angle>-3.14159</min_angle>
+            <max_angle>3.14159</max_angle>
+          </horizontal>
+          <vertical>
+            <samples>16</samples>
+            <resolution>1</resolution>
+            <min_angle>-0.261799</min_angle>
+            <max_angle>0.261799</max_angle>
+          </vertical>
+        </scan>
+        <range>
+          <min>0.1</min>
+          <max>100.0</max>
+          <resolution>0.01</resolution>
+        </range>
+      </lidar>
+      <visualize>false</visualize>
+    </sensor>
+  </gazebo>
+  <!-- IMU -->
+  <gazebo reference="imu_link">
+    <sensor name="imu_sensor" type="imu">
+      <topic>imu/data</topic>
+      <update_rate>100</update_rate>
+      <gz_frame_id>imu_link</gz_frame_id>
+      <always_on>true</always_on>
+    </sensor>
+  </gazebo>
 </robot>

Commit message: feat: crawler telemetry/protection, IK test env, multi-camera support
crawler_driver:
- Full Roboclaw telemetry reading (current, speed, temp, voltage, status)
- Hardware current limit via SETM1/M2MAXCURRENT on startup
- Velocity-error-based stall detection with output scaling
- 9 diagnostics topics under ~/diagnostics/

bringup:
- launch_config.yaml for enabling/disabling subsystems at launch time
- cameras.yaml: YAML-driven multi-camera config (v4l2 + RealSense)
- camera.launch.py: iterate cameras.yaml, per-camera container + QR opt-in
- ffmpeg_to_foxglove_video.py: configurable input/output topics
- test_ik.launch.py: IK test environment without real hardware
- arm_mock_driver.py: joint state feedback loop for IK testing
- arm_teleop.py: keyboard teleop for arm Cartesian + gripper
- Justfile: nixGL support, display/ik/teleop-arm recipes

urdf:
- Add gripper_joint7/8 to robot.urdf.xacro and sekirei.urdf

qr_detector:
- Use relative topic names for namespace-based multi-camera routing

Co-Authored-By: Claude Sonnet 4.6 <noreply@anthropic.com>

File: main_ws/src/bringup/urdf/robot.urdf.xacro (robot description, xacro)
@@ -118,4 +118,21 @@
     <origin xyz="0.15 0 ${base_height/2 + 0.05}"/>
   </joint>
+  <!-- Gripper (parallel link, 2x Dynamixel) -->
+  <link name="gripper_left_link"/>
+  <link name="gripper_right_link"/>
+  <joint name="gripper_joint7" type="revolute">
+    <origin xyz="0 0 0"/>
+    <axis xyz="0 1 0"/>
+    <parent link="arm6_link"/>
+    <child link="gripper_left_link"/>
+    <limit effort="5" lower="-1.57" upper="1.57" velocity="1.0"/>
+  </joint>
+  <joint name="gripper_joint8" type="revolute">
+    <origin xyz="0 0 0"/>
+    <axis xyz="0 1 0"/>
+    <parent link="arm6_link"/>
+    <child link="gripper_right_link"/>
+    <limit effort="5" lower="-1.57" upper="1.57" velocity="1.0"/>
+  </joint>
   <link name="imu_link"/>
   <joint name="imu_joint" type="fixed">

File: main_ws/src/bringup/urdf/sekirei.urdf (robot description, URDF)
Before this commit: robot sekirei, 11 links, 10 joints
Links:
- added link gripper_left_link
- added link gripper_right_link
Joints:
- added joint gripper_joint7: type revolute, parent arm6_link, child gripper_left_link, origin xyz=0 0 0 rpy=0 0 0, axis 0 1 0, limit lower=-1.57 upper=1.57 effort=5 velocity=1.0
- added joint gripper_joint8: type revolute, parent arm6_link, child gripper_right_link, origin xyz=0 0 0 rpy=0 0 0, axis 0 1 0, limit lower=-1.57 upper=1.57 effort=5 velocity=1.0

Commit message: fix(perception): resolve TF conflict and fix laserscan queue overflow
Three related issues:
- pointcloud_to_laserscan was dropping all messages because target_frame
  "base_footprint" required a multi-hop TF lookup that filled the
  MessageFilter queue immediately. Changed to "base_link" which is
  resolved directly via URDF static TF.
- lidar_static_tf (static_transform_publisher) and robot_state_publisher
  were both publishing base_link→velodyne, creating a TF race condition.
  Removed lidar_static_tf; URDF velodyne_joint is now the sole authority.
- Updated velodyne_joint origin from (0.15, 0, 0.125) to (0, 0, 0) to
  match the real-robot calibration that lidar_static_tf was enforcing.

Co-Authored-By: Claude Sonnet 4.6 <noreply@anthropic.com>

File: main_ws/src/bringup/urdf/robot.urdf.xacro (robot description, xacro)
@@ -132,5 +132,5 @@
     <parent link="base_link"/>
     <child link="velodyne"/>
-    <origin xyz="0.15 0 ${base_height/2 + 0.05}"/>
+    <origin xyz="0 0 0"/>
   </joint>
   <!-- Gripper (parallel link, 2x Dynamixel) -->

Commit message: refactor(crawler_driver): serial I/O を専用スレッドに分離、効率改善
- serial スレッド導入: すべての Roboclaw I/O を専用スレッドに移動
  - ROS executor スレッドが serial ブロックで止まらなくなった
  - watchdog / telemetry タイマーが serial I/O 中でも確実に発火する
  - 接続・再接続も serial スレッドが自律的に処理
- コマンドスロット (latest-wins): cmd_vel は最新指令のみ保持
- Mixed Speed コマンド (cmd=37): M1+M2 を1トランザクションで原子送信
  - 左右タイミングずれ解消、serial 往復コスト半減
- heap alloc ゼロ: Packet 構造体 (stack 固定 32bytes) で vector を置き換え
- stall 検出を telemetry 周期 (10Hz) に固定: dt が安定
- cmd_vel=0 振動対策: 停止遷移時のみ stop コマンド送信、以降は沈黙
- Kd=0.008 追加: PI 積分残留による停止時振動を減衰
- flipper: wheel mode 設定直後に goalVelocity=0 送信 (再起動後の暴走防止)
- odom_selector: T265 切り替え時の SE(3) オフセット補償で位置ジャンプを防止
- nav2_params: D435i depth → /scan_depth 観測ソースを local_costmap に追加
- urdf: 6台 v4l2 カメラの TF リンクを追加 (Foxglove 3D 表示修正)
- system.launch: use_nav2=true かつ use_lidar=false の不整合を起動時に警告
- control.launch: RSP 二重起動バグを修正 (robot_description 競合解消)

Co-Authored-By: Claude Sonnet 4.6 <noreply@anthropic.com>

File: main_ws/src/bringup/urdf/robot.urdf.xacro (robot description, xacro)
@@ -162,4 +162,83 @@
     <child link="imu_link"/>
     <origin xyz="0 0 0"/>
+  </joint>
+  <!-- ======================== RealSense Cameras ======================== -->
+  <!--
+    FIXME: 以下の xyz / rpy は仮値。実機でノギス等を使って計測し調整すること。
+    realsense2_camera が publish する base_frame_id はこれらのリンク名と一致させている。
+    シリアル番号は `rs-enumerate-devices` で確認し cameras.yaml に設定すること。
+  -->
+  <!-- RealSense T265 (トラッキングカメラ)
+       マウント位置: arm_base_link の右側面 (-y 方向)、ロボット後方向き
+       rpy = "0 -pi/2 0" により T265 の +z (光軸) が base_link の -x (後方) を向く -->
+  <link name="camera_t265_link">
+    <visual>
+      <geometry><mesh filename="package://bringup/meshes/t265.STL" scale="${mesh_scale}"/></geometry>
+      <material name="silver"/>
+    </visual>
+    <xacro:dummy_inertial/>
+  </link>
+  <joint name="camera_t265_joint" type="fixed">
+    <parent link="arm_base_link"/>
+    <child link="camera_t265_link"/>
+    <!-- xyz: arm_base_link から右 5cm・上 2cm。rpy: 後方向き (-90° pitch) -->
+    <origin xyz="0.0 -0.05 0.02" rpy="0 ${-pi/2} 0"/>
+  </joint>
+  <!-- RealSense D435i (RGB-D カメラ)
+       マウント位置: arm6_link (エンドエフェクタ) の左側面 (+y 方向)、グリッパと同方向
+       arm6_link の向きはアーム姿勢依存なので rpy は 0 0 0 で出発し実機で確認すること -->
+  <link name="camera_d435i_link">
+    <visual>
+      <geometry><mesh filename="package://bringup/meshes/d435.STL" scale="${mesh_scale}"/></geometry>
+      <material name="silver"/>
+    </visual>
+    <xacro:dummy_inertial/>
+  </link>
+  <joint name="camera_d435i_joint" type="fixed">
+    <parent link="arm6_link"/>
+    <child link="camera_d435i_link"/>
+    <!-- xyz: arm6_link から左 4cm。グリッパと同じ方向を向く -->
+    <origin xyz="0.0 0.04 0.0" rpy="0 0 0"/>
+  </joint>
+  <!-- ======================== v4l2 カメラ TF リンク ======================== -->
+  <!--
+    FIXME: 以下の xyz / rpy は仮値。実機でノギス等を使って計測し調整すること。
+    TF ツリーに接続されていないと Foxglove の 3D 表示・QR 検出位置マッピングが壊れる。
+  -->
+  <!-- フロントカメラ: 前面中央、前向き -->
+  <link name="front_camera_link"><xacro:dummy_inertial/></link>
+  <joint name="front_camera_joint" type="fixed">
+    <parent link="base_link"/><child link="front_camera_link"/>
+    <origin xyz="${base_length/2} 0 ${base_height/2 + 0.02}" rpy="0 0 0"/>
+  </joint>
+  <!-- バックカメラ: 後面中央、後向き -->
+  <link name="back_camera_link"><xacro:dummy_inertial/></link>
+  <joint name="back_camera_joint" type="fixed">
+    <parent link="base_link"/><child link="back_camera_link"/>
+    <origin xyz="${-base_length/2} 0 ${base_height/2 + 0.02}" rpy="0 0 ${pi}"/>
+  </joint>
+  <!-- 左カメラ: 左側面、左向き -->
+  <link name="left_camera_link"><xacro:dummy_inertial/></link>
+  <joint name="left_camera_joint" type="fixed">
+    <parent link="base_link"/><child link="left_camera_link"/>
+    <origin xyz="0 ${base_width/2} ${base_height/2 + 0.02}" rpy="0 0 ${pi/2}"/>
+  </joint>
+  <!-- 右カメラ: 右側面、右向き -->
+  <link name="right_camera_link"><xacro:dummy_inertial/></link>
+  <joint name="right_camera_joint" type="fixed">
+    <parent link="base_link"/><child link="right_camera_link"/>
+    <origin xyz="0 ${-base_width/2} ${base_height/2 + 0.02}" rpy="0 0 ${-pi/2}"/>
+  </joint>
+  <!-- アームカメラ: arm_base_link 前方の汎用 USB カメラ -->
+  <link name="arm_camera_link"><xacro:dummy_inertial/></link>
+  <joint name="arm_camera_joint" type="fixed">
+    <parent link="arm_base_link"/><child link="arm_camera_link"/>
+    <origin xyz="0.05 0 0.05" rpy="0 0 0"/>
+  </joint>
+  <!-- THETA S: 天板中央、360° カメラ -->
+  <link name="theta_camera_link"><xacro:dummy_inertial/></link>
+  <joint name="theta_camera_joint" type="fixed">
+    <parent link="base_link"/><child link="theta_camera_link"/>
+    <origin xyz="0 0 ${base_height/2 + 0.10}" rpy="0 0 0"/>
   </joint>
   <!-- ======================== Gazebo Plugins ======================== -->
