Commit message: today's work

File: main_ws/src/bringup/urdf/robot.urdf.xacro (robot description, xacro)
@@ -176,5 +176,5 @@
       <visual>
         <geometry>
-          <mesh filename="package://arm_controller/meshes/flipper.STL"/>
+          <mesh filename="package://bringup/meshes/flipper.STL"/>
         </geometry>
         <origin xyz="0 0 0" rpy="${flip_rpy}"/>
@@ -190,5 +190,5 @@
     </link>
     <joint name="${name}_joint" type="revolute">
-      <origin xyz="${x_offset} ${y_offset} 0.06" rpy="0 0 0"/>
+      <origin xyz="${x_offset} ${y_offset} ${-base_height/2}" rpy="0 0 0"/>
       <axis xyz="0 1 0"/>
       <parent link="base_link"/>
@@ -202,13 +202,16 @@
     </gazebo>
   </xacro:macro>
-  <!-- 前方: x = -base_length/2 付近, 後方: x = +base_length/2 付近 -->
-  <xacro:flipper name="flipper_fr" x_offset="-0.2135" y_offset="0.205"  flip_rpy="0 0 1.57"/>
-  <xacro:flipper name="flipper_fl" x_offset="-0.2135" y_offset="-0.205" flip_rpy="0 0 -1.57"/>
-  <xacro:flipper name="flipper_br" x_offset="0.2135"  y_offset="0.205"  flip_rpy="0 0 1.57"/>
-  <xacro:flipper name="flipper_bl" x_offset="0.2135"  y_offset="-0.205" flip_rpy="0 0 -1.57"/>
+  <!-- 前方 (+X = カメラ側): base_length/2, 後方 (-X = アーム側): -base_length/2 -->
+  <!-- flipper.STL は Z 方向に 0.28m 伸びる。pitch ±90° で水平に倒す。  -->
+  <!-- 前方: pitch +90° → Z_mesh → +X_robot (前方に伸びる) -->
+  <!-- 後方: pitch -90° → Z_mesh → -X_robot (後方に伸びる) -->
+  <xacro:flipper name="flipper_fr" x_offset="${base_length/2}"  y_offset="${track_width/2}"   flip_rpy="0 ${pi/2} 0"/>
+  <xacro:flipper name="flipper_fl" x_offset="${base_length/2}"  y_offset="${-track_width/2}"  flip_rpy="0 ${pi/2} 0"/>
+  <xacro:flipper name="flipper_br" x_offset="${-base_length/2}" y_offset="${track_width/2}"   flip_rpy="0 ${-pi/2} 0"/>
+  <xacro:flipper name="flipper_bl" x_offset="${-base_length/2}" y_offset="${-track_width/2}"  flip_rpy="0 ${-pi/2} 0"/>
   <!-- ======================== 6DOF Arm (sekirei URDF 由来) ======================== -->
   <!--
     arm_controller の sekirei.urdf をシミュ用に再構成。
-    Visual: 実機と同じ STL メッシュ (package://arm_controller/meshes/)
+    Visual: 実機と同じ STL メッシュ (package://bringup/meshes/)
     Collision: 簡易ボックスで軽量化
     Inertia: 各リンク 0.5 kg 均一近似
@@ -217,5 +220,5 @@
   <link name="arm_base_link">
     <visual>
-      <geometry><mesh filename="package://arm_controller/meshes/r_a_2019_2020_asm1.STL"/></geometry>
+      <geometry><mesh filename="package://bringup/meshes/r_a_2019_2020_asm1.STL"/></geometry>
       <origin xyz="-0.08 -0.081 0" rpy="1.57 0 0"/>
       <material name="white"><color rgba="1 1 1 1"/></material>
@@ -234,5 +237,5 @@
   <link name="arm1_link">
     <visual>
-      <geometry><mesh filename="package://arm_controller/meshes/r_a_2019_2020_asm2.STL"/></geometry>
+      <geometry><mesh filename="package://bringup/meshes/r_a_2019_2020_asm2.STL"/></geometry>
       <origin xyz="0 0 0.004" rpy="1.57 0 0"/>
       <material name="white"><color rgba="1 1 1 1"/></material>
@@ -255,5 +258,5 @@
   <link name="arm2_link">
     <visual>
-      <geometry><mesh filename="package://arm_controller/meshes/r_a_2019_2020_asm3.STL"/></geometry>
+      <geometry><mesh filename="package://bringup/meshes/r_a_2019_2020_asm3.STL"/></geometry>
       <origin xyz="0 0 0" rpy="1.57 0 0"/>
       <material name="white"><color rgba="1 1 1 1"/></material>
@@ -276,5 +279,5 @@
   <link name="arm3_link">
     <visual>
-      <geometry><mesh filename="package://arm_controller/meshes/r_a_2019_2020_asm4.STL"/></geometry>
+      <geometry><mesh filename="package://bringup/meshes/r_a_2019_2020_asm4.STL"/></geometry>
       <origin xyz="0 0 0" rpy="1.57 0 0"/>
       <material name="white"><color rgba="1 1 1 1"/></material>
@@ -297,5 +300,5 @@
   <link name="arm4_link">
     <visual>
-      <geometry><mesh filename="package://arm_controller/meshes/r_a_2019_2020_asm5.STL"/></geometry>
+      <geometry><mesh filename="package://bringup/meshes/r_a_2019_2020_asm5.STL"/></geometry>
       <origin xyz="0 0 0" rpy="1.57 3.14 0"/>
       <material name="white"><color rgba="1 1 1 1"/></material>
@@ -317,5 +320,5 @@
   <link name="arm5_link">
     <visual>
-      <geometry><mesh filename="package://arm_controller/meshes/r_a_2019_l_asm6.STL"/></geometry>
+      <geometry><mesh filename="package://bringup/meshes/r_a_2019_l_asm6.STL"/></geometry>
       <origin xyz="0 0 0" rpy="1.57 3.14 0"/>
       <material name="white"><color rgba="1 1 1 1"/></material>
@@ -337,5 +340,5 @@
   <link name="arm6_link">
     <visual>
-      <geometry><mesh filename="package://arm_controller/meshes/r_a_2019_l_asm7_ver2.STL"/></geometry>
+      <geometry><mesh filename="package://bringup/meshes/r_a_2019_l_asm7_ver2.STL"/></geometry>
       <origin xyz="0 0 0" rpy="0 3.14 0"/>
       <material name="white"><color rgba="1 1 1 1"/></material>

Commit message: model fixed

File: main_ws/src/bringup/urdf/robot.urdf.xacro (robot description, xacro)
@@ -202,12 +202,14 @@
     </gazebo>
   </xacro:macro>
-  <!-- 前方 (+X = カメラ側): base_length/2, 後方 (-X = アーム側): -base_length/2 -->
-  <!-- flipper.STL は Z 方向に 0.28m 伸びる。pitch ±90° で水平に倒す。  -->
-  <!-- 前方: pitch +90° → Z_mesh → +X_robot (前方に伸びる) -->
-  <!-- 後方: pitch -90° → Z_mesh → -X_robot (後方に伸びる) -->
-  <xacro:flipper name="flipper_fr" x_offset="${base_length/2}"  y_offset="${track_width/2}"   flip_rpy="0 ${pi/2} 0"/>
-  <xacro:flipper name="flipper_fl" x_offset="${base_length/2}"  y_offset="${-track_width/2}"  flip_rpy="0 ${pi/2} 0"/>
-  <xacro:flipper name="flipper_br" x_offset="${-base_length/2}" y_offset="${track_width/2}"   flip_rpy="0 ${-pi/2} 0"/>
-  <xacro:flipper name="flipper_bl" x_offset="${-base_length/2}" y_offset="${-track_width/2}"  flip_rpy="0 ${-pi/2} 0"/>
+  <!--
+    flipper.STL 座標系: X=厚み(8.3cm), Y=幅(11cm), Z=長さ(28cm, +Z方向)
+    roll+yaw の組み合わせで (mesh X,Y,Z) → (robot Z,X/Y,Z→X) に変換。
+    FR/BR: 厚み→+Y (右外側),  FL/BL: 厚み→-Y (左外側)
+    FR/FL: 長さ→+X (前方),    BR/BL: 長さ→-X (後方)
+  -->
+  <xacro:flipper name="flipper_fr" x_offset="${base_length/2}"  y_offset="${track_width/2}"   flip_rpy="${pi/2} 0 ${pi/2}"/>
+  <xacro:flipper name="flipper_fl" x_offset="${base_length/2}"  y_offset="${-track_width/2}"  flip_rpy="${-pi/2} 0 ${-pi/2}"/>
+  <xacro:flipper name="flipper_br" x_offset="${-base_length/2}" y_offset="${track_width/2}"   flip_rpy="${-pi/2} 0 ${pi/2}"/>
+  <xacro:flipper name="flipper_bl" x_offset="${-base_length/2}" y_offset="${-track_width/2}"  flip_rpy="${pi/2} 0 ${-pi/2}"/>
   <!-- ======================== 6DOF Arm (sekirei URDF 由来) ======================== -->
   <!--
@@ -230,5 +232,5 @@
   </link>
   <joint name="arm_base_link_joint" type="fixed">
-    <origin xyz="-0.2 0 ${base_height/2 + 0.02}" rpy="0 0 0"/>
+    <origin xyz="-0.2 0 ${base_height/2 + 0.06}" rpy="0 0 0"/>
     <parent link="base_link"/>
     <child link="arm_base_link"/>

File: main_ws/src/bringup/urdf/sekirei.urdf (robot description, URDF)
Before this commit: robot sekirei, 11 links, 10 joints
Links:
- link arm1_link: geometry visual mesh filename=package://bringup/meshes/r_a_2019_2020_asm2.STL
- link arm2_link: geometry visual mesh filename=package://bringup/meshes/r_a_2019_2020_asm3.STL
- link arm3_link: geometry visual mesh filename=package://bringup/meshes/r_a_2019_2020_asm4.STL
- link arm4_link: geometry visual mesh filename=package://bringup/meshes/r_a_2019_2020_asm5.STL
- link arm5_link: geometry visual mesh filename=package://bringup/meshes/r_a_2019_l_asm6.STL
- link arm6_link: geometry visual mesh filename=package://bringup/meshes/r_a_2019_l_asm7_ver2.STL
- link arm_base_link: geometry visual mesh filename=package://bringup/meshes/r_a_2019_2020_asm1.STL
- link gui_d435_link: geometry visual mesh filename=package://bringup/meshes/d435.STL
- link gui_t265_link: geometry visual mesh filename=package://bringup/meshes/t265.STL

Commit message: fix: Gazeboシミュレーション安定化 & teleop追加
URDF:
- preserveFixedJoint追加 (caster/velodyne/imu/camera/arm_base/tip)
- アーム関節: effort/damping/PID大幅強化 (重力補償)
- フリッパーPID強化 (p=50, i=0.5, d=15)
- self_collide=false追加

Launch:
- GZ_SIM_RESOURCE_PATH設定 (メッシュ解決)
- --render-engine ogre (Nix環境Vulkan非対応対策)
- odom_tf_bridge追加 (odom→base_footprint TF)

新規:
- odom_tf_bridge.py: /odom→TF broadcaster
- teleop-twist-keyboard: flake.nixに追加

修正:
- arm_gz_bridge.py: 二重shutdown回避
- simulation.rviz: Fixed Frame=base_link (TF解決待ち問題回避)

File: main_ws/src/bringup/urdf/robot.urdf.xacro (robot description, xacro)
@@ -112,4 +112,7 @@
     <child link="caster_link"/>
   </joint>
+  <gazebo reference="caster_joint">
+    <preserveFixedJoint>true</preserveFixedJoint>
+  </gazebo>
   <!-- ======================== VLP-16 LiDAR ======================== -->
   <link name="velodyne">
@@ -132,4 +135,7 @@
     <child link="velodyne"/>
   </joint>
+  <gazebo reference="velodyne_joint">
+    <preserveFixedJoint>true</preserveFixedJoint>
+  </gazebo>
   <!-- ======================== IMU ======================== -->
   <link name="imu_link">
@@ -145,4 +151,7 @@
     <child link="imu_link"/>
   </joint>
+  <gazebo reference="imu_joint">
+    <preserveFixedJoint>true</preserveFixedJoint>
+  </gazebo>
   <!-- ======================== Camera ======================== -->
   <link name="camera_link">
@@ -165,4 +174,7 @@
     <child link="camera_link"/>
   </joint>
+  <gazebo reference="camera_joint">
+    <preserveFixedJoint>true</preserveFixedJoint>
+  </gazebo>
   <!-- ======================== Flippers (sekirei_workspace 由来) ======================== -->
   <!--
@@ -236,4 +248,7 @@
     <child link="arm_base_link"/>
   </joint>
+  <gazebo reference="arm_base_link_joint">
+    <preserveFixedJoint>true</preserveFixedJoint>
+  </gazebo>
   <!-- Joint 1: 旋回 (Z 軸) -->
   <link name="arm1_link">
@@ -254,6 +269,6 @@
     <parent link="arm_base_link"/>
     <child link="arm1_link"/>
-    <limit effort="5" lower="-3.14" upper="3.14" velocity="1.571"/>
-    <dynamics damping="0.3" friction="0.1"/>
+    <limit effort="10" lower="-3.14" upper="3.14" velocity="1.571"/>
+    <dynamics damping="1.0" friction="0.2"/>
   </joint>
   <!-- Joint 2: 肩 (Y 軸) -->
@@ -275,6 +290,6 @@
     <parent link="arm1_link"/>
     <child link="arm2_link"/>
-    <limit effort="5" lower="-3.14" upper="0" velocity="1.571"/>
-    <dynamics damping="0.3" friction="0.1"/>
+    <limit effort="20" lower="-3.14" upper="0" velocity="1.571"/>
+    <dynamics damping="2.0" friction="0.3"/>
   </joint>
   <!-- Joint 3: 肘 (Y 軸) -->
@@ -296,6 +311,6 @@
     <parent link="arm2_link"/>
     <child link="arm3_link"/>
-    <limit effort="5" lower="0" upper="3.14" velocity="1.571"/>
-    <dynamics damping="0.3" friction="0.1"/>
+    <limit effort="20" lower="0" upper="3.14" velocity="1.571"/>
+    <dynamics damping="2.0" friction="0.3"/>
   </joint>
   <!-- Joint 4: 手首ピッチ (Y 軸) -->
@@ -316,6 +331,6 @@
     <parent link="arm3_link"/>
     <child link="arm4_link"/>
-    <limit effort="5" lower="-4.71" upper="0" velocity="1.571"/>
-    <dynamics damping="0.2" friction="0.1"/>
+    <limit effort="10" lower="-4.71" upper="0" velocity="1.571"/>
+    <dynamics damping="1.0" friction="0.2"/>
   </joint>
   <!-- Joint 5: 手首ヨー (Z 軸) -->
@@ -337,5 +352,5 @@
     <child link="arm5_link"/>
     <limit effort="5" lower="-1.57" upper="1.57" velocity="1.571"/>
-    <dynamics damping="0.2" friction="0.1"/>
+    <dynamics damping="0.5" friction="0.1"/>
   </joint>
   <!-- Joint 6: 手首ロール (X 軸) -->
@@ -357,5 +372,5 @@
     <child link="arm6_link"/>
     <limit effort="5" lower="-3.14" upper="3.14" velocity="1.571"/>
-    <dynamics damping="0.2" friction="0.1"/>
+    <dynamics damping="0.5" friction="0.1"/>
   </joint>
   <!-- End effector (tip) -->
@@ -372,7 +387,14 @@
     <child link="link_tip"/>
   </joint>
+  <gazebo reference="tip_joint">
+    <preserveFixedJoint>true</preserveFixedJoint>
+  </gazebo>
   <!-- ============================================================ -->
   <!--                Gazebo Harmonic (gz sim) Plugins              -->
   <!-- ============================================================ -->
+  <!-- モデルレベル: 自己衝突無効化 -->
+  <gazebo reference="base_link">
+    <self_collide>false</self_collide>
+  </gazebo>
   <!-- Differential Drive (クローラの近似) -->
   <gazebo>
@@ -505,7 +527,7 @@
       <joint_name>flipper_fr_joint</joint_name>
       <topic>flipper_fr_joint/cmd_pos</topic>
-      <p_gain>20</p_gain>
-      <i_gain>0</i_gain>
-      <d_gain>5</d_gain>
+      <p_gain>50</p_gain>
+      <i_gain>0.5</i_gain>
+      <d_gain>15</d_gain>
     </plugin>
     <plugin filename="gz-sim-joint-position-controller-system"
@@ -513,7 +535,7 @@
       <joint_name>flipper_fl_joint</joint_name>
       <topic>flipper_fl_joint/cmd_pos</topic>
-      <p_gain>20</p_gain>
-      <i_gain>0</i_gain>
-      <d_gain>5</d_gain>
+      <p_gain>50</p_gain>
+      <i_gain>0.5</i_gain>
+      <d_gain>15</d_gain>
     </plugin>
     <plugin filename="gz-sim-joint-position-controller-system"
@@ -521,7 +543,7 @@
       <joint_name>flipper_br_joint</joint_name>
       <topic>flipper_br_joint/cmd_pos</topic>
-      <p_gain>20</p_gain>
-      <i_gain>0</i_gain>
-      <d_gain>5</d_gain>
+      <p_gain>50</p_gain>
+      <i_gain>0.5</i_gain>
+      <d_gain>15</d_gain>
     </plugin>
     <plugin filename="gz-sim-joint-position-controller-system"
@@ -529,10 +551,10 @@
       <joint_name>flipper_bl_joint</joint_name>
       <topic>flipper_bl_joint/cmd_pos</topic>
-      <p_gain>20</p_gain>
-      <i_gain>0</i_gain>
-      <d_gain>5</d_gain>
-    </plugin>
-  </gazebo>
-  <!-- Arm joints の位置制御 -->
+      <p_gain>50</p_gain>
+      <i_gain>0.5</i_gain>
+      <d_gain>15</d_gain>
+    </plugin>
+  </gazebo>
+  <!-- Arm joints の位置制御 (重力補償のため高ゲイン) -->
   <gazebo>
     <plugin filename="gz-sim-joint-position-controller-system"
@@ -540,5 +562,6 @@
       <joint_name>arm_joint1</joint_name>
       <topic>arm_joint1/cmd_pos</topic>
-      <p_gain>30</p_gain><i_gain>0</i_gain><d_gain>8</d_gain>
+      <p_gain>100</p_gain><i_gain>2</i_gain><d_gain>20</d_gain>
+      <cmd_max>50</cmd_max><cmd_min>-50</cmd_min>
     </plugin>
     <plugin filename="gz-sim-joint-position-controller-system"
@@ -546,5 +569,6 @@
       <joint_name>arm_joint2</joint_name>
       <topic>arm_joint2/cmd_pos</topic>
-      <p_gain>30</p_gain><i_gain>0</i_gain><d_gain>8</d_gain>
+      <p_gain>150</p_gain><i_gain>5</i_gain><d_gain>30</d_gain>
+      <cmd_max>80</cmd_max><cmd_min>-80</cmd_min>
     </plugin>
     <plugin filename="gz-sim-joint-position-controller-system"
@@ -552,5 +576,6 @@
       <joint_name>arm_joint3</joint_name>
       <topic>arm_joint3/cmd_pos</topic>
-      <p_gain>30</p_gain><i_gain>0</i_gain><d_gain>8</d_gain>
+      <p_gain>150</p_gain><i_gain>5</i_gain><d_gain>30</d_gain>
+      <cmd_max>80</cmd_max><cmd_min>-80</cmd_min>
     </plugin>
     <plugin filename="gz-sim-joint-position-controller-system"
@@ -558,5 +583,6 @@
       <joint_name>arm_joint4</joint_name>
       <topic>arm_joint4/cmd_pos</topic>
-      <p_gain>30</p_gain><i_gain>0</i_gain><d_gain>8</d_gain>
+      <p_gain>100</p_gain><i_gain>2</i_gain><d_gain>20</d_gain>
+      <cmd_max>50</cmd_max><cmd_min>-50</cmd_min>
     </plugin>
     <plugin filename="gz-sim-joint-position-controller-system"
@@ -564,5 +590,6 @@
       <joint_name>arm_joint5</joint_name>
       <topic>arm_joint5/cmd_pos</topic>
-      <p_gain>30</p_gain><i_gain>0</i_gain><d_gain>8</d_gain>
+      <p_gain>60</p_gain><i_gain>1</i_gain><d_gain>12</d_gain>
+      <cmd_max>30</cmd_max><cmd_min>-30</cmd_min>
     </plugin>
     <plugin filename="gz-sim-joint-position-controller-system"
@@ -570,5 +597,6 @@
       <joint_name>arm_joint6</joint_name>
       <topic>arm_joint6/cmd_pos</topic>
-      <p_gain>30</p_gain><i_gain>0</i_gain><d_gain>8</d_gain>
+      <p_gain>60</p_gain><i_gain>1</i_gain><d_gain>12</d_gain>
+      <cmd_max>30</cmd_max><cmd_min>-30</cmd_min>
     </plugin>
   </gazebo>
