Commit message: arm

File: main_ws/src/bringup/urdf/robot.urdf.xacro (robot description, xacro)
@@ -62,30 +62,30 @@
     <xacro:dummy_inertial/>
   </link>
-  <joint name="arm_joint1" type="revolute"><origin xyz="0 0 0"/><axis xyz="0 0 1"/><parent link="arm_base_link"/><child link="arm1_link"/><limit effort="10" lower="-3.14" upper="3.14" velocity="1.571"/></joint>
+  <joint name="arm_joint1" type="revolute"><origin xyz="0 0 0"/><axis xyz="0 0 1"/><parent link="arm_base_link"/><child link="arm1_link"/><limit effort="10" lower="-6.28" upper="6.28" velocity="1.571"/></joint>
   <link name="arm2_link">
     <visual><origin xyz="0 0 0" rpy="1.57 0 0"/><geometry><mesh filename="package://bringup/meshes/r_a_2019_2020_asm3.STL" scale="${mesh_scale}"/></geometry></visual>
     <xacro:dummy_inertial/>
   </link>
-  <joint name="arm_joint2" type="revolute"><origin xyz="0 -0.048 0.078"/><axis xyz="0 1 0"/><parent link="arm1_link"/><child link="arm2_link"/><limit effort="20" lower="-3.14" upper="0" velocity="1.571"/></joint>
+  <joint name="arm_joint2" type="revolute"><origin xyz="0 -0.048 0.078"/><axis xyz="0 1 0"/><parent link="arm1_link"/><child link="arm2_link"/><limit effort="20" lower="-6.28" upper="0" velocity="1.571"/></joint>
   <link name="arm3_link">
     <visual><origin xyz="0 0 0" rpy="1.57 0 0"/><geometry><mesh filename="package://bringup/meshes/r_a_2019_2020_asm4.STL" scale="${mesh_scale}"/></geometry></visual>
     <xacro:dummy_inertial/>
   </link>
-  <joint name="arm_joint3" type="revolute"><origin xyz="0.45 0.007 0.084"/><axis xyz="0 1 0"/><parent link="arm2_link"/><child link="arm3_link"/><limit effort="20" lower="0" upper="3.14" velocity="1.571"/></joint>
+  <joint name="arm_joint3" type="revolute"><origin xyz="0.45 0.007 0.084"/><axis xyz="0 1 0"/><parent link="arm2_link"/><child link="arm3_link"/><limit effort="20" lower="-6.28" upper="6.28" velocity="1.571"/></joint>
   <link name="arm4_link">
     <visual><origin xyz="0 0 0" rpy="1.57 3.14 0"/><geometry><mesh filename="package://bringup/meshes/r_a_2019_2020_asm5.STL" scale="${mesh_scale}"/></geometry></visual>
     <xacro:dummy_inertial/>
   </link>
-  <joint name="arm_joint4" type="revolute"><origin xyz="-0.5 0.012 0"/><axis xyz="0 1 0"/><parent link="arm3_link"/><child link="arm4_link"/><limit effort="10" lower="-4.71" upper="0" velocity="1.571"/></joint>
+  <joint name="arm_joint4" type="revolute"><origin xyz="-0.5 0.012 0"/><axis xyz="0 1 0"/><parent link="arm3_link"/><child link="arm4_link"/><limit effort="10" lower="-6.28" upper="6.28" velocity="1.571"/></joint>
   <link name="arm5_link">
     <visual><origin xyz="0 0 0" rpy="1.57 3.14 0"/><geometry><mesh filename="package://bringup/meshes/r_a_2019_l_asm6.STL" scale="${mesh_scale}"/></geometry></visual>
     <xacro:dummy_inertial/>
   </link>
-  <joint name="arm_joint5" type="revolute"><origin xyz="0.06525 0.028 0.029647"/><axis xyz="0 0 1"/><parent link="arm4_link"/><child link="arm5_link"/><limit effort="5" lower="-1.57" upper="1.57" velocity="1.571"/></joint>
+  <joint name="arm_joint5" type="revolute"><origin xyz="0.06525 0.028 0.029647"/><axis xyz="0 0 1"/><parent link="arm4_link"/><child link="arm5_link"/><limit effort="5" lower="-3.14" upper="3.14" velocity="1.571"/></joint>
   <link name="arm6_link">
     <visual><origin xyz="0 0 0" rpy="0 3.14 0"/><geometry><mesh filename="package://bringup/meshes/r_a_2019_l_asm7_ver2.STL" scale="${mesh_scale}"/></geometry></visual>
     <xacro:dummy_inertial/>
   </link>
-  <joint name="arm_joint6" type="revolute"><origin xyz="0.07425 0 -0.03"/><axis xyz="1 0 0"/><parent link="arm5_link"/><child link="arm6_link"/><limit effort="5" lower="-3.14" upper="3.14" velocity="1.571"/></joint>
+  <joint name="arm_joint6" type="revolute"><origin xyz="0.07425 0 -0.03"/><axis xyz="1 0 0"/><parent link="arm5_link"/><child link="arm6_link"/><limit effort="5" lower="-6.28" upper="6.28" velocity="1.571"/></joint>
   <!-- ======================== Simulation: Drive Wheels ======================== -->
   <!-- クローラを diff_drive で近似する仮想ホイール (シミュレーション専用) -->

File: main_ws/src/bringup/urdf/sekirei.urdf (robot description, URDF)
Before this commit: robot sekirei, 13 links, 12 joints
Joints:
- joint arm_joint1: limit lower=-3.14 upper=3.14 effort=5 velocity=1.571 -> lower=-6.28 upper=6.28 effort=5 velocity=1.571
- joint arm_joint2: limit lower=-3.14 upper=0 effort=5 velocity=1.571 -> lower=-6.28 upper=0 effort=5 velocity=1.571
- joint arm_joint3: limit lower=-0.72 upper=3.14 effort=5 velocity=1.571 -> lower=-6.28 upper=6.28 effort=5 velocity=1.571
- joint arm_joint4: limit lower=-4.71 upper=0 effort=5 velocity=1.571 -> lower=-6.28 upper=6.28 effort=5 velocity=1.571
- joint arm_joint5: limit lower=-1.57 upper=1.57 effort=5 velocity=1.571 -> lower=-3.14 upper=3.14 effort=5 velocity=1.571
- joint arm_joint6: limit lower=-3.14 upper=3.14 effort=5 velocity=1.571 -> lower=-6.28 upper=6.28 effort=5 velocity=1.571

File: main_ws/src/control/moveit/urdf/sekirei_moveit.xacro (robot description, xacro)
@@ -105,5 +105,5 @@
   <joint name="arm_joint3" type="revolute">
     <origin xyz="0.45 0.007 0.084" rpy="0 0 0"/>
-    <axis xyz="0 -1 0"/>
+    <axis xyz="0 1 0"/>
     <parent link="arm2_link"/>
     <child link="arm3_link"/>
